File: elektryczny/PUEE.kicad_pcb (KiCad board)
At the start: 2 copper layers, 62 parts, among them J1 CAN, J2 VIN, J3 OLED, J4 Button1, J5 LED1, J6 Button1, J7 Conn_01x05, J8 Conn_01x07, SW1 Button2, SW2 Button1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

Commit message: update
Parts:
- removed J3: OLED, Connector_PinHeader_2.54mm:PinHeader_1x04_P2.54mm_Vertical
- removed J4, J6: Button1, Connector_PinHeader_2.54mm:PinHeader_1x03_P2.54mm_Vertical
- removed J5: LED1, Connector_PinHeader_2.54mm:PinHeader_1x03_P2.54mm_Vertical
- removed J8: Conn_01x07, Connector_PinHeader_2.54mm:PinHeader_1x07_P2.54mm_Vertical
- C3: value 100nF -> 10nF
- C4: value 100nF -> 1uF
- J7: value Conn_01x05 -> STM
- U3: footprint Package_SO:Texas_HSOP-8-1EP_3.9x4.9mm_P1.27mm -> Package_TO_SOT_SMD:SOT-23-6
- moved R5 74.9 mm to (126.6, 41.9), turned to 90 degrees
- moved R4 72.0 mm to (124.6, 41.9), turned to 90 degrees
- moved C7 64.8 mm to (175.8, 89.8), turned to 90 degrees
- moved R6 63.2 mm to (128.6, 41.9), turned to 90 degrees
- moved C11 62.8 mm to (147.6, 51.6)
- moved C6 62.4 mm to (175.8, 98.3), turned to 90 degrees
- moved C12 62.0 mm to (156.4, 50.9)
- moved R11 60.7 mm to (169.0, 54.0), turned to -90 degrees
- moved Y2 58.3 mm to (171.4, 96.6), turned to 90 degrees
- moved U11 57.9 mm to (143.5, 126.6), turned to 90 degrees
- moved R13 56.7 mm to (152.2, 56.5)
- moved U10 56.7 mm to (143.5, 118.7), turned to 90 degrees
- moved U13 56.0 mm to (163.0, 54.0)
- moved R12 55.9 mm to (152.2, 54.5)
- moved U9 55.3 mm to (143.5, 110.7), turned to 90 degrees
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
Commit message: poprawki pcb
Parts:
- moved R4 81.1 mm to (161.0, 114.3), turned to -90 degrees
- moved R5 79.4 mm to (159.0, 114.3), turned to -90 degrees
- moved R6 77.8 mm to (157.0, 114.3), turned to -90 degrees
- moved U11 75.4 mm to (129.1, 52.6), turned to -90 degrees
- moved C22 74.3 mm to (124.3, 54.5), turned to 90 degrees
- moved U2 67.4 mm to (165.5, 103.0), turned to -90 degrees
- moved C8 63.2 mm to (171.5, 91.4), turned to -90 degrees
- moved U10 60.0 mm to (129.1, 60.5), turned to -90 degrees
- moved C21 59.3 mm to (124.3, 62.5), turned to 90 degrees
- moved R2 58.7 mm to (169.0, 91.4), turned to -90 degrees
- moved R3 51.7 mm to (165.0, 91.4), turned to -90 degrees
- moved C20 45.1 mm to (124.3, 70.5), turned to 90 degrees
- moved U9 44.6 mm to (129.1, 68.5), turned to -90 degrees
- moved C10 36.1 mm to (154.2, 92.2), turned to 0 degrees
- moved C13 34.6 mm to (117.7, 67.0), turned to 90 degrees
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