File: elektryczny/PUEE — kopia.kicad_pcb (KiCad board)
At the start: 2 copper layers, 57 parts, among them J1 CAN, J2 VIN, J7 STM, SW1 Button2, SW2 Button1, U1 STM32F042F4Px, U10 WS2815, U11 WS2815, U13 SN65HVD230QDRG4Q1, U2 ESP-12E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

Commit message: polaczenia pcb czesc 1/2
Parts:
- C1: moved to F.Cu
- moved C13 22.6 mm to (117.7, 67.0)
- moved R10 19.2 mm to (119.3, 50.2)
- moved C14 19.2 mm to (121.2, 60.6)
- moved R8 19.2 mm to (117.8, 60.6)
- moved SW1 19.2 mm to (119.4, 72.5)
- moved SW2 19.2 mm to (119.5, 55.0)
- moved R9 19.0 mm to (119.5, 77.2), turned to 0 degrees
- moved R7 15.7 mm to (121.2, 66.9)
- moved U4 8.74 mm to (136.5, 53.0)
- moved C16 8.73 mm to (140.8, 62.8)
- moved U5 8.73 mm to (136.5, 60.8)
- moved C15 8.73 mm to (140.8, 54.7)
- moved C18 8.73 mm to (140.8, 78.2)
- moved U7 8.73 mm to (136.5, 76.2)
- moved C17 8.73 mm to (140.8, 70.5)
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Connections:
- C11 pad 1: -12V -> +12V
- C11 pad 2: +12V -> -12V
- R11 pad 1: /CAN_L -> /CAN_H
- R11 pad 2: /CAN_H -> /CAN_L
Routing:
- net -12V: track 248.1 -> 16.2 mm, vias 4 -> 0
- net +12V: track 137.4 -> 0.00 mm, vias 1 -> 0
- net VDD: track 162.8 -> 58.5 mm, vias 3 -> 0
- net /SPI1_NSS: track 45.6 -> 0.00 mm, vias 2 -> 0
- net /GPIO_Button1: track 35.4 -> 0.00 mm
- net /GPIO_Button2: track 29.4 -> 0.00 mm
- net Net-(U3-FB): track 21.7 -> 0.00 mm, vias 1 -> 0
- net Net-(U3-SW): track 21.1 -> 0.00 mm
- net Net-(R10-Pad2): track 15.3 -> 0.00 mm
- net Net-(R7-Pad1): track 15.2 -> 0.00 mm
- net /USART2_RX: track 12.3 -> 0.00 mm
- net Net-(U7-DO): track 12.2 -> 0.00 mm
- net /NRST: track 14.4 -> 5.29 mm
- net /USART2_TX: track 8.57 -> 0.00 mm
- net /CAN_H: track 7.62 -> 0.00 mm
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
Commit message: polaczenia attempt 1, do poprawki
Parts:
- moved C1 6.16 mm to (149.4, 77.0)
- moved C2 6.16 mm to (151.6, 77.0)
- moved U1 5.36 mm to (158.5, 77.5)
Routing:
- net VDD: track 58.5 -> 0.00 mm
- net Net-(U1-PF0): track 17.8 -> 0.00 mm
- net -12V: track 16.2 -> 0.00 mm
- net Net-(C6-Pad1): track 10.8 -> 0.00 mm
- net VDDA: track 8.74 -> 0.00 mm
- net Net-(U4-NC): track 7.03 -> 0.00 mm
- net Net-(U7-NC): track 7.03 -> 0.00 mm
- net Net-(U5-NC): track 7.00 -> 0.00 mm
- net Net-(U6-NC): track 6.97 -> 0.00 mm
- net Net-(U9-NC): track 6.81 -> 0.00 mm
- net Net-(U11-NC): track 6.77 -> 0.00 mm
- net Net-(U10-NC): track 6.77 -> 0.00 mm
- net Net-(U8-NC): track 6.73 -> 0.00 mm
- net Net-(U2-~{RST}): track 5.59 -> 0.00 mm
- net /NRST: track 5.29 -> 0.00 mm
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